File: 8b.kicad_pcb (KiCad board)
At the start: 2 copper layers, 61 parts, among them J1 AudioJack2, J11 AudioJack3, J2 AudioJack2, J3 AudioJack2, J4 AudioJack2, J5 AudioJack2, J6 AudioJack2, J7 AudioJack2, J8 AudioJack2, J9 AudioJack3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

Commit message: Update footprint components
Parts:
- D1: footprint ArcadeButtons:sanwa-obsf-30-g -> Diode_THT:D_DO-35_SOD27_P7.62mm_Horizontal
Changed lines of the file:
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@@
     )
   )
-  (footprint "ArcadeButtons:sanwa-obsf-30-g" (layer "F.Cu")
+  (footprint "Diode_THT:D_DO-35_SOD27_P7.62mm_Horizontal" (layer "F.Cu")
     (at 87.207829 73.213458)
+    (descr "Diode, DO-35_SOD27 series, Axial, Horizontal, pin pitch=7.62mm, , length*diameter=4*2mm^2, , http://www.diodes.com/_files/packages/DO-35.pdf")
+    (tags "Diode DO-35_SOD27 series Axial Horizontal pin pitch 7.62mm  length 4mm diameter 2mm")
     (property "Sheetfile" "8b.kicad_sch")
     (property "Sheetname" "")
@@
     (property "ki_keywords" "diode")
     (attr through_hole)
-    (fp_text reference "D1" (at 0 -0.5 unlocked) (layer "F.SilkS")
-        (effects (font (size 1 1) (thickness 0.1)))
-    )
-    (fp_text value "1N4148" (at 0 7.62 unlocked) (layer "F.Fab")
+    (fp_text reference "D1" (at 3.81 -2.12) (layer "F.SilkS")
         (effects (font (size 1 1) (thickness 0.15)))
     )
-    (fp_text user "${REFERENCE}" (at 0 10.16 unlocked) (layer "F.Fab")
+    (fp_text value "1N4148" (at 3.81 2.12) (layer "F.Fab")
         (effects (font (size 1 1) (thickness 0.15)))
     )
-    (fp_rect (start -10.16 -10.16) (end 10.16 5.08)
-      (stroke (width 0.2) (type default)) (fill none) (layer "F.SilkS"))
-    (fp_circle (center 0 -2.985629) (end 19.067829 -2.985629)
-      (stroke (width 0.05) (type default)) (fill none) (layer "F.CrtYd"))
-    (pad "1" thru_hole oval (at -4.7105 0) (size 2 5) (drill oval 1 3.5) (layers "*.Cu" "*.Mask")
+    (fp_text user "K" (at 0 -1.8) (layer "F.SilkS")
+        (effects (font (size 1 1) (thickness 0.15)))
+    )
+    (fp_text user "K" (at 0 -1.8) (layer "F.Fab")
+        (effects (font (size 1 1) (thickness 0.15)))
+    )
+    (fp_text user "${REFERENCE}" (at 4.11 0) (layer "F.Fab")
+        (effects (font (size 0.8 0.8) (thickness 0.12)))
+    )
+    (fp_line (start 1.04 0) (end 1.69 0)
+      (stroke (width 0.12) (type solid)) (layer "F.SilkS"))
+    (fp_line (start 1.69 -1.12) (end 1.69 1.12)
+      (stroke (width 0.12) (type solid)) (layer "F.SilkS"))
+    (fp_line (start 1.69 1.12) (end 5.93 1.12)
+      (stroke (width 0.12) (type solid)) (layer "F.SilkS"))
+    (fp_line (start 2.29 -1.12) (end 2.29 1.12)
+      (stroke (width 0.12) (type solid)) (layer "F.SilkS"))
+    (fp_line (start 2.41 -1.12) (end 2.41 1.12)
+      (stroke (width 0.12) (type solid)) (layer "F.SilkS"))
+    (fp_line (start 2.53 -1.12) (end 2.53 1.12)
+      (stroke (width 0.12) (type solid)) (layer "F.SilkS"))
+    (fp_line (start 5.93 -1.12) (end 1.69 -1.12)
+      (stroke (width 0.12) (type solid)) (layer "F.SilkS"))
+    (fp_line (start 5.93 1.12) (end 5.93 -1.12)
+      (stroke (width 0.12) (type solid)) (layer "F.SilkS"))
+    (fp_line (start 6.58 0) (end 5.93 0)
+      (stroke (width 0.12) (type solid)) (layer "F.SilkS"))
+    (fp_line (start -1.05 -1.25) (end -1.05 1.25)
+      (stroke (width 0.05) (type solid)) (layer "F.CrtYd"))
+    (fp_line (start -1.05 1.25) (end 8.67 1.25)
+      (stroke (width 0.05) (type solid)) (layer "F.CrtYd"))
+    (fp_line (start 8.67 -1.25) (end -1.05 -1.25)
+      (stroke (width 0.05) (type solid)) (layer "F.CrtYd"))
+    (fp_line (start 8.67 1.25) (end 8.67 -1.25)
+      (stroke (width 0.05) (type solid)) (layer "F.CrtYd"))
+    (fp_line (start 0 0) (end 1.81 0)
+      (stroke (width 0.1) (type solid)) (layer "F.Fab"))
+    (fp_line (start 1.81 -1) (end 1.81 1)
+      (stroke (width 0.1) (type solid)) (layer "F.Fab"))
+    (fp_line (start 1.81 1) (end 5.81 1)
+      (stroke (width 0.1) (type solid)) (layer "F.Fab"))
+    (fp_line (start 2.31 -1) (end 2.31 1)
+      (stroke (width 0.1) (type solid)) (layer "F.Fab"))
+    (fp_line (start 2.41 -1) (end 2.41 1)
+      (stroke (width 0.1) (type solid)) (layer "F.Fab"))
+    (fp_line (start 2.51 -1) (end 2.51 1)
+      (stroke (width 0.1) (type solid)) (layer "F.Fab"))
+    (fp_line (start 5.81 -1) (end 1.81 -1)
+      (stroke (width 0.1) (type solid)) (layer "F.Fab"))
+    (fp_line (start 5.81 1) (end 5.81 -1)
+      (stroke (width 0.1) (type solid)) (layer "F.Fab"))
+    (fp_line (start 7.62 0) (end 5.81 0)
+      (stroke (width 0.1) (type solid)) (layer "F.Fab"))
+    (pad "1" thru_hole rect (at 0 0) (size 1.6 1.6) (drill 0.8) (layers "*.Cu" "*.Mask")
       (net 1 "+3.3V") (pinfunction "K") (pintype "passive"))
-    (pad "2" thru_hole oval (at 4.7105 0) (size 2 5) (drill oval 1 3.5) (layers "*.Cu" "*.Mask")
+    (pad "2" thru_hole oval (at 7.62 0) (size 1.6 1.6) (drill 0.8) (layers "*.Cu" "*.Mask")
       (net 2 "/SCL") (pinfunction "A") (pintype "passive"))
-    (model "${KIPRJMOD}/lib/kicad-lib/3dmodels/sanwa obsf-30-g.STEP"
-      (offset (xyz 11.85 5 12.5))
+    (model "${KICAD6_3DMODEL_DIR}/Diode_THT.3dshapes/D_DO-35_SOD27_P7.62mm_Horizontal.wrl"
+      (offset (xyz 0 0 0))
       (scale (xyz 1 1 1))
-      (rotate (xyz -90 0 0))
+      (rotate (xyz 0 0 0))
     )
   )

Commit message: Layout draft
Parts:
- moved J9 192.9 mm to (274.3, 130.4), turned to 90 degrees
- moved R9 161.6 mm to (52.9, 48.0)
- moved R10 160.9 mm to (70.0, 31.9), turned to -90 degrees
- moved U1 160.3 mm to (46.4, 131.4), turned to 90 degrees
- moved J1 154.7 mm to (60.0, 23.2)
- moved Q1 153.2 mm to (70.0, 49.3), turned to 90 degrees
- moved Q2 139.3 mm to (95.0, 49.3), turned to 90 degrees
- moved R11 135.3 mm to (77.9, 48.0)
- moved R12 131.1 mm to (95.0, 31.9), turned to -90 degrees
- moved Q3 123.2 mm to (120.0, 49.3), turned to 90 degrees
- moved J11 118.5 mm to (103.6, 147.2), turned to 0 degrees
- moved R14 117.9 mm to (120.0, 31.9), turned to -90 degrees
- moved R13 117.6 mm to (102.9, 48.0)
- moved J2 116.7 mm to (85.0, 23.2)
- moved Q4 115.3 mm to (145.0, 49.3), turned to 90 degrees
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Other:
- board outline added: 254 x 125 mm
